File: hw/rev-a/gb-link-usb.kicad_sch (KiCad schematic)
At the start: 41 parts, among them SW1 434133025816, SW2 434133025816, U1 RP2350A, U2 NCP1117ST33T3G, U3 W25Q128JVSIQ, X1 12MHz

Commit message: PCB rev A routed: scripted build + Freerouting pipeline, DRC 0 errors
Co-Authored-By: Claude Opus 5.5 (1M context) <noreply@anthropic.com>
Claude-Session: https://claude.ai/code/session_01MZ3uQJCcn6FcjzVDhZnLJN
Parts:
- removed MH1, MH2, MH3, MH4: NPTH FD2.75mm SM3.15mm KO6mm, RPI_COMPILED:none_mh_npth_fd2p75mm_sm3p15mm_ko6mm, symbol RPI_DB:Mechanical | Mounting_Holes/RP-01HF5R-LCTEJS
Connections:
- net GPIO11: now reaches U1.15 (GPIO11)
- net GPIO12: now reaches U1.16 (GPIO12)
- net GPIO13: now reaches U1.17 (GPIO13)
- net GPIO14: now reaches U1.18 (GPIO14)
- net GPIO21: now reaches U1.33 (GPIO21)
- net GPIO0: no longer names the net of U1.2 (GPIO0)
- net GPIO1: no longer names the net of U1.3 (GPIO1)
- net GPIO2: no longer names the net of U1.4 (GPIO2)
- net GPIO25: no longer names the net of U1.37 (GPIO25)
- net GPIO3: no longer names the net of U1.5 (GPIO3)
- net SWCLK: no longer names the net of U1.24 (SWCLK)
- net SWD: no longer names the net of U1.25 (SWDIO)
- no-connect marks 25 -> 27

Commit message: PCB rev A: JLC order files (BOM, CPL, Gerbers, pin audit), core LCSC parts
Not ordered. Hold point: L1 (AOTA-B201610S3R3-101-T) has 4 in JLC stock.
LED pad numbering fixed in the CPL (JLC A=1, KiCad K=1).

Co-Authored-By: Claude Opus 5.5 (1M context) <noreply@anthropic.com>
Claude-Session: https://claude.ai/code/session_01MZ3uQJCcn6FcjzVDhZnLJN
Parts:
- C1, C19, C5: LCSC (none) -> C15850
- C10, C11, C12, C13, C14, C15, C16, C17, C18, C2, C8: LCSC (none) -> C1525
- C3, C4: LCSC (none) -> C1548
- C6, C7, C9: LCSC (none) -> C23733
- L1: value 3.3u -> AOTA-B201610S3R3-101-T; LCSC (none) -> C42411119
- PCB1, SBREV1, VARIANT1: now left out of the parts list
- R1: LCSC (none) -> C25744
- R10: LCSC (none) -> C17168
- R2, R4, R6: LCSC (none) -> C11702
- R3: LCSC (none) -> C25105
- R7, R8: LCSC (none) -> C25100
- SW1, SW2: value 434133025816 -> SKRPABE010; LCSC (none) -> C115360
- U1: LCSC (none) -> C42411118
- U2: LCSC (none) -> C26537
- U3: LCSC (none) -> C97521
- X1: value 12MHz -> ABM8-272-T3; LCSC (none) -> C20625731
